File: Automatic Changeover.sch (EAGLE design)
At the start: 49 parts, among them IC1 ACS750LCA-050, IC2 XMEGA16A4A, IC4 ACS750LCA-050, IC5 ACS750LCA-050, K1 S216SE1, K2 S216SE1, K3 S216SE1, K4 S216SE1, K5 S216SE1, K6 S216SE1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

Commit message: almost done--just trace with of high DC current left
Changed lines of the file:
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@@
 <wire x1="53.34" y1="25.4" x2="53.34" y2="27.94" width="0.1524" layer="91"/>
 <junction x="53.34" y="25.4"/>
+<label x="50.8" y="22.86" size="1.778" layer="95"/>
 </segment>
 </net>
@@
 <segment>
 <pinref part="B3" gate="1" pin="AC2"/>
-<wire x1="-63.5" y1="76.2" x2="-63.5" y2="73.66" width="0.1524" layer="91"/>
-<wire x1="-63.5" y1="73.66" x2="-137.16" y2="73.66" width="0.1524" layer="91"/>
-<label x="-149.86" y="73.66" size="1.778" layer="95"/>
-</segment>
-<segment>
+<wire x1="-63.5" y1="76.2" x2="-63.5" y2="78.74" width="0.1524" layer="91"/>
+<wire x1="-63.5" y1="78.74" x2="-137.16" y2="78.74" width="0.1524" layer="91"/>
+<label x="-152.4" y="78.74" size="1.778" layer="95"/>
+</segment>
+<segment>
